File: LanguageCard.kicad_pcb (KiCad board)
At the start: 2 copper layers, 100 x 77.5 mm, 44 parts, among them J1 Apple II Expansion Bus, SW1 ROM ENABLE, U1 74LS86, U10 74LS06, U2 74LS08, U3 74LS175, U4 74LS32, U5 74LS08, U6 74LS08, U7 ROM F8 (2716/32)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

Commit message: rev 3
Parts:
- removed C10, C11: 100n, Capacitor_THT:C_Disc_D3.0mm_W1.6mm_P2.50mm
- C2, C3, C4, C5, C6, C7, C8, C9: footprint Capacitor_THT:C_Disc_D3.0mm_W1.6mm_P2.50mm -> Capacitor_THT:C_Axial_L3.8mm_D2.6mm_P7.50mm_Horizontal
- moved C4 62.0 mm to (95.8, 41.9)
- moved C7 53.7 mm to (88.3, 87.6), turned to 0 degrees
- moved C3 52.8 mm to (144.8, 36.8), turned to 90 degrees
- moved C5 51.7 mm to (131.4, 54.7), turned to -90 degrees
- moved C8 47.7 mm to (131.4, 81.2), turned to 90 degrees
- moved C9 44.0 mm to (154.3, 81.2)
- moved C6 22.8 mm to (154.3, 54.7), turned to -90 degrees
- moved C2 5.04 mm to (116.8, 36.8)
Routing:
- net +5V: track 4.45 -> 29.1 mm
- net GND: track 19.7 -> 42.8 mm
- net /ABNK: track 47.0 -> 48.6 mm
- net /A3: track 119.9 -> 121.5 mm
- net /A13: track 96.4 -> 97.7 mm
- net Net-(R6-Pad1): track 54.2 -> 55.5 mm
- net /A1: track 165.2 -> 166.6 mm
- net Net-(U5-Pad2): track 30.7 -> 31.9 mm
- net Net-(U2-Pad1): track 41.5 -> 40.3 mm
- net /ROMA11/VPP/~{WE}: track 56.3 -> 55.4 mm
- net /~{RESET}: track 28.2 -> 29.0 mm
- net /~{A13}: track 153.7 -> 154.5 mm
- net /WE: track 111.3 -> 112.1 mm
