File: LanguageCard.kicad_sch (KiCad schematic)
At the start: 39 parts, among them J1 Apple II Expansion Bus, SW1 ROM ENABLE, U1 74LS86, U10 74LS06, U2 74LS08, U3 74LS175, U4 74LS32, U5 74LS08, U6 74LS08, U7 ROM F8 (2716/32)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

Commit message: rev 3
Parts:
- removed C10, C11: 100n, Capacitor_THT:C_Disc_D3.0mm_W1.6mm_P2.50mm, symbol Device:C
- C2, C3, C4, C5, C6, C7, C8, C9: footprint Capacitor_THT:C_Disc_D3.0mm_W1.6mm_P2.50mm -> Capacitor_THT:C_Axial_L3.8mm_D2.6mm_P7.50mm_Horizontal
Changed lines of the file:
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@@
   (paper "USLegal")
   (title_block
-    (date "2023-08-30")
-    (rev "2")
-  )
-  (junction (at 234.95 19.05) (diameter 0) (color 0 0 0 0)
+    (date "2023-09-21")
+    (rev "3")
   )
   (junction (at 66.04 76.2) (diameter 0) (color 0 0 0 0)
@@
   (junction (at 218.44 96.52) (diameter 0) (color 0 0 0 0)
   )
-  (junction (at 86.36 83.82) (diameter 0) (color 0 0 0 0)
+  (junction (at 234.95 26.67) (diameter 0) (color 0 0 0 0)
   )
-  (junction (at 250.19 19.05) (diameter 0) (color 0 0 0 0)
+  (junction (at 86.36 83.82) (diameter 0) (color 0 0 0 0)
   )
   (junction (at 196.85 19.05) (diameter 0) (color 0 0 0 0)
@@
   (junction (at 304.8 81.28) (diameter 0) (color 0 0 0 0)
   )
-  (junction (at 250.19 26.67) (diameter 0) (color 0 0 0 0)
-  )
   (junction (at 212.09 19.05) (diameter 0) (color 0 0 0 0)
   )
   (junction (at 227.33 19.05) (diameter 0) (color 0 0 0 0)
   )
+  (junction (at 234.95 19.05) (diameter 0) (color 0 0 0 0)
+  )
   (junction (at 124.46 110.49) (diameter 0) (color 0 0 0 0)
   )
@@
   (junction (at 49.53 129.54) (diameter 0) (color 0 0 0 0)
   )
-  (junction (at 234.95 26.67) (diameter 0) (color 0 0 0 0)
-  )
   (junction (at 34.29 68.58) (diameter 0) (color 0 0 0 0)
   )
@@
   (junction (at 227.33 26.67) (diameter 0) (color 0 0 0 0)
   )
-  (junction (at 242.57 19.05) (diameter 0) (color 0 0 0 0)
-  )
   (junction (at 219.71 19.05) (diameter 0) (color 0 0 0 0)
   )
@@
   (junction (at 288.29 114.3) (diameter 0) (color 0 0 0 0)
   )
-  (junction (at 242.57 26.67) (diameter 0) (color 0 0 0 0)
-  )
   (junction (at 204.47 26.67) (diameter 0) (color 0 0 0 0)
   )
@@
     (stroke (width 0) (type default))
   )
+  (wire (pts (xy 234.95 26.67) (xy 242.57 26.67))
+    (stroke (width 0) (type default))
+  )
   (wire (pts (xy 34.29 68.58) (xy 34.29 71.12))
     (stroke (width 0) (type default))
@@
     (stroke (width 0) (type default))
   )
-  (wire (pts (xy 250.19 19.05) (xy 242.57 19.05))
-    (stroke (width 0) (type default))
-  )
   (wire (pts (xy 219.71 26.67) (xy 212.09 26.67))
     (stroke (width 0) (type default))
@@
     (stroke (width 0) (type default))
   )
-  (wire (pts (xy 250.19 26.67) (xy 257.81 26.67))
-    (stroke (width 0) (type default))
-  )
-  (wire (pts (xy 242.57 19.05) (xy 234.95 19.05))
-    (stroke (width 0) (type default))
-  )
   (wire (pts (xy 25.4 153.67) (xy 33.02 153.67))
     (stroke (width 0) (type default))
@@
     (stroke (width 0) (type default))
   )
-  (wire (pts (xy 250.19 26.67) (xy 242.57 26.67))
-    (stroke (width 0) (type default))
-  )
   (wire (pts (xy 91.44 40.64) (xy 91.44 30.48))
     (stroke (width 0) (type default))
@@
     (stroke (width 0) (type default))
   )
-  (wire (pts (xy 242.57 26.67) (xy 234.95 26.67))
-    (stroke (width 0) (type default))
-  )
   (wire (pts (xy 193.04 67.31) (xy 200.66 67.31))
     (stroke (width 0) (type default))
@@
     (stroke (width 0) (type default))
   )
+  (wire (pts (xy 234.95 19.05) (xy 242.57 19.05))
+    (stroke (width 0) (type default))
+  )
   (wire (pts (xy 25.4 27.94) (xy 68.58 27.94))
     (stroke (width 0) (type default))
@@
     (stroke (width 0) (type default))
   )
-  (wire (pts (xy 250.19 19.05) (xy 257.81 19.05))
-    (stroke (width 0) (type default))
-  )
   (wire (pts (xy 132.08 35.56) (xy 134.62 35.56))
     (stroke (width 0) (type default))
@@
       (effects (font (size 1.27 1.27)) (justify right))
     )
-    (property "Footprint" "Capacitor_THT:C_Disc_D3.0mm_W1.6mm_P2.50mm" (at 211.1248 26.67 0)
+    (property "Footprint" "Capacitor_THT:C_Axial_L3.8mm_D2.6mm_P7.50mm_Horizontal" (at 211.1248 26.67 0)
       (effects (font (size 1.27 1.27)) hide)
     )
@@
     )
   )
+  (symbol (lib_id "Device:C") (at 242.57 22.86 0) (mirror y) (unit 1)
+    (in_bom yes) (on_board yes) (dnp no)
+    (property "Reference" "C9" (at 242.57 20.32 0)
+      (effects (font (size 1.27 1.27)) (justify right))
+    )
+    (property "Value" "100n" (at 242.57 25.4 0)
+      (effects (font (size 1.27 1.27)) (justify right))
+    )
+    (property "Footprint" "Capacitor_THT:C_Axial_L3.8mm_D2.6mm_P7.50mm_Horizontal" (at 241.6048 26.67 0)
+      (effects (font (size 1.27 1.27)) hide)
+    )
+    (property "Datasheet" "~" (at 242.57 22.86 0)
+      (effects (font (size 1.27 1.27)) hide)
+    )
+    (pin "1")
+    (pin "2")
+    (instances
+      (project "LanguageCard"
+        (path "/e35c56f9-4713-4571-acdb-6ae2f2073fad"
+          (reference "C9") (unit 1)
+        )
+      )
+    )
+  )
   (symbol (lib_id "power:+5V") (at 204.47 124.46 0) (unit 1)
     (in_bom yes) (on_board yes) (dnp no) (fields_autoplaced)
@@
     )
   )
-  (symbol (lib_id "Device:C") (at 242.57 22.86 0) (mirror y) (unit 1)
-    (in_bom yes) (on_board yes) (dnp no)
-    (property "Reference" "C9" (at 242.57 20.32 0)
-      (effects (font (size 1.27 1.27)) (justify right))
-    )
-    (property "Value" "100n" (at 242.57 25.4 0)
-      (effects (font (size 1.27 1.27)) (justify right))
-    )
-    (property "Footprint" "Capacitor_THT:C_Disc_D3.0mm_W1.6mm_P2.50mm" (at 241.6048 26.67 0)
-      (effects (font (size 1.27 1.27)) hide)
-    )
-    (property "Datasheet" "~" (at 242.57 22.86 0)
-      (effects (font (size 1.27 1.27)) hide)
-    )
-    (pin "1")
-    (pin "2")
-    (instances
-      (project "LanguageCard"
-        (path "/e35c56f9-4713-4571-acdb-6ae2f2073fad"
-          (reference "C9") (unit 1)
-        )
-      )
-    )
-  )
   (symbol (lib_id "74xx:74LS06") (at 40.64 129.54 0) (unit 6)
     (in_bom yes) (on_board yes) (dnp no) (fields_autoplaced)
@@
       (effects (font (size 1.27 1.27)) (justify right))
     )
-    (property "Footprint" "Capacitor_THT:C_Disc_D3.0mm_W1.6mm_P2.50mm" (at 203.5048 26.67 0)
+    (property "Footprint" "Capacitor_THT:C_Axial_L3.8mm_D2.6mm_P7.50mm_Horizontal" (at 203.5048 26.67 0)
       (effects (font (size 1.27 1.27)) hide)
     )
@@
     )
   )
-  (symbol (lib_id "Device:C") (at 257.81 22.86 0) (mirror y) (unit 1)
-    (in_bom yes) (on_board yes) (dnp no)
-    (property "Reference" "C11" (at 257.81 20.32 0)
-      (effects (font (size 1.27 1.27)) (justify right))
-    )
-    (property "Value" "100n" (at 257.81 25.4 0)
-      (effects (font (size 1.27 1.27)) (justify right))
-    )
-    (property "Footprint" "Capacitor_THT:C_Disc_D3.0mm_W1.6mm_P2.50mm" (at 256.8448 26.67 0)
-      (effects (font (size 1.27 1.27)) hide)
-    )
-    (property "Datasheet" "~" (at 257.81 22.86 0)
-      (effects (font (size 1.27 1.27)) hide)
-    )
-    (pin "1")
-    (pin "2")
-    (instances
-      (project "LanguageCard"
-        (path "/e35c56f9-4713-4571-acdb-6ae2f2073fad"
-          (reference "C11") (unit 1)
-        )
-      )
-    )
-  )
   (symbol (lib_id "74xx:74LS86") (at 68.58 66.04 0) (unit 3)
     (in_bom yes) (on_board yes) (dnp no) (fields_autoplaced)
@@
       (effects (font (size 1.27 1.27)) (justify right))
     )
-    (property "Footprint" "Capacitor_THT:C_Disc_D3.0mm_W1.6mm_P2.50mm" (at 195.8848 19.05 0)
+    (property "Footprint" "Capacitor_THT:C_Axial_L3.8mm_D2.6mm_P7.50mm_Horizontal" (at 195.8848 19.05 0)
       (effects (font (size 1.27 1.27)) hide)
     )
@@
       (effects (font (size 1.27 1.27)) (justify right))
     )
-    (property "Footprint" "Capacitor_THT:C_Disc_D3.0mm_W1.6mm_P2.50mm" (at 188.2648 19.05 0)
+    (property "Footprint" "Capacitor_THT:C_Axial_L3.8mm_D2.6mm_P7.50mm_Horizontal" (at 188.2648 19.05 0)
       (effects (font (size 1.27 1.27)) hide)
     )
@@
       (effects (font (size 1.27 1.27)) (justify right))
     )
-    (property "Footprint" "Capacitor_THT:C_Disc_D3.0mm_W1.6mm_P2.50mm" (at 233.9848 26.67 0)
+    (property "Footprint" "Capacitor_THT:C_Axial_L3.8mm_D2.6mm_P7.50mm_Horizontal" (at 233.9848 26.67 0)
       (effects (font (size 1.27 1.27)) hide)
     )
@@
       (effects (font (size 1.27 1.27)) (justify right))
     )
-    (property "Footprint" "Capacitor_THT:C_Disc_D3.0mm_W1.6mm_P2.50mm" (at 218.7448 26.67 0)
+    (property "Footprint" "Capacitor_THT:C_Axial_L3.8mm_D2.6mm_P7.50mm_Horizontal" (at 218.7448 26.67 0)
       (effects (font (size 1.27 1.27)) hide)
     )
@@
     )
   )
-  (symbol (lib_id "Device:C") (at 250.19 22.86 0) (mirror y) (unit 1)
-    (in_bom yes) (on_board yes) (dnp no)
-    (property "Reference" "C10" (at 250.19 20.32 0)
-      (effects (font (size 1.27 1.27)) (justify right))
-    )
-    (property "Value" "100n" (at 250.19 25.4 0)
-      (effects (font (size 1.27 1.27)) (justify right))
-    )
-    (property "Footprint" "Capacitor_THT:C_Disc_D3.0mm_W1.6mm_P2.50mm" (at 249.2248 26.67 0)
-      (effects (font (size 1.27 1.27)) hide)
-    )
-    (property "Datasheet" "~" (at 250.19 22.86 0)
-      (effects (font (size 1.27 1.27)) hide)
-    )
-    (pin "1")
-    (pin "2")
-    (instances
-      (project "LanguageCard"
-        (path "/e35c56f9-4713-4571-acdb-6ae2f2073fad"
-          (reference "C10") (unit 1)
-        )
-      )
-    )
-  )
   (symbol (lib_id "Device:C_Polarized_US") (at 124.46 135.89 0) (unit 1)
     (in_bom yes) (on_board yes) (dnp no) (fields_autoplaced)
@@
       (effects (font (size 1.27 1.27)) (justify right))
     )
-    (property "Footprint" "Capacitor_THT:C_Disc_D3.0mm_W1.6mm_P2.50mm" (at 226.3648 26.67 0)
+    (property "Footprint" "Capacitor_THT:C_Axial_L3.8mm_D2.6mm_P7.50mm_Horizontal" (at 226.3648 26.67 0)
       (effects (font (size 1.27 1.27)) hide)
     )
